File: airSensor_V1.kicad_sch (KiCad schematic)
At the start: 27 parts, among them J1 USB_C_Receptacle_USB2.0_14P, J2 Conn_01x04_Socket, SW1 SW_Push, SW2 SW_Push, SW3 SW_Push, U1 ESP32-C3-WROOM-02, U2 AP2112K-3.3, U3 SHT4x, U4 SGP40-D-R4

Commit message: Initial commit for air sensor project
Parts:
- removed D2: LED, LED_SMD:LED_0805_2012Metric, symbol Device:LED
- added C10: 100nf, Capacitor_SMD:C_0805_2012Metric, symbol Device:C_Small
- added C11, C8: 100nF, Capacitor_SMD:C_0805_2012Metric, symbol Device:C_Small
- added C9: 10uf, Capacitor_SMD:C_0805_2012Metric, symbol Device:C_Small
- added J3: Conn_01x02_Socket, Resistor_SMD:R_0805_2012Metric, symbol Connector:Conn_01x02_Socket
- added R10: 2k, Resistor_SMD:R_0805_2012Metric, symbol Device:R
- added SW4: SW_Push, Button_Switch_THT:SW_PUSH_6mm, symbol Switch:SW_Push
- added SW5: SW_SPDT, Button_Switch_THT:SW_Slide_SPDT_Straight_CK_OS102011MS2Q, symbol Switch:SW_SPDT
- added U5: MCP73831-2-OT, Package_TO_SOT_SMD:SOT-23-5, symbol Battery_Management:MCP73831-2-OT
- added U6: SCD40-D-R2, Sensor:Sensirion_SCD4x-1EP_10.1x10.1mm_P1.25mm_EP4.8x4.8mm, symbol Sensor_Gas:SCD40-D-R2
- R9: value 330 -> 10k
Connections:
- net +3.3V: now also R9.1, C11.1, U6.19 (VDD), U6.7 (VDD)
- net GND: now also C10.2, C11.2, C8.2, C9.1, J3.2 (Pin_2), R10.2, SW4.2, U5.2 (V_{SS}), U6.20 (GND), U6.21 (GND), U6.6 (GND)
- net I2C_SCL: now also U6.9 (SCL)
- net I2C_SDA: now also U6.10 (SDA)
- net IO18: now also J1.A7 (D-), J1.B7 (D-); no longer J1.A6 (D+), J1.B6 (D+)
- net IO19: now also J1.A6 (D+), J1.B6 (D+); no longer J1.A7 (D-), J1.B7 (D-)
- net Read_User: now reaches R9.2
- net Read_User: now also U1.3 (IO4), C8.1, SW4.1
- net +5V renamed USB_IN
- net USB_IN: now also C9.2, U5.4 (V_{DD}); no longer C4.1, U2.1 (VIN), U2.3 (EN)
- removed net IO4: R9.1, U1.3 (IO4)
- new net: R10.1, U5.5 (PROG)
- new net BATT: C10.1, J3.1 (Pin_1), SW5.1 (A), U5.3 (V_{BAT})
- new net VSYS: C4.1, SW5.2 (B), U2.1 (VIN), U2.3 (EN)
- no-connect marks 1 -> 3
Other:
- moved on the sheet: D1, R7, SW1, SW2, SW3
