File: airSensor_V1.kicad_pcb (KiCad board)
At the start: 2 copper layers, 27 parts, among them J1 USB_C_Receptacle_USB2.0_14P, J2 Conn_01x04_Socket, SW1 SW_Push, SW2 SW_Push, SW3 SW_Push, U1 ESP32-C3-WROOM-02, U2 AP2112K-3.3, U3 SHT4x, U4 SGP40-D-R4

Commit message: Initial commit for air sensor project
Parts:
- added C10: 100nf, Capacitor_SMD:C_0805_2012Metric, F.Cu at (149.7, 87.0)
- added C11: 100nF, Capacitor_SMD:C_0805_2012Metric, F.Cu at (149.7, 90.0)
- added C4: 10uf, Capacitor_SMD:C_0805_2012Metric, F.Cu at (149.7, 78.0)
- added C8: 100nF, Capacitor_SMD:C_0805_2012Metric, F.Cu at (149.7, 81.0)
- added C9: 10uf, Capacitor_SMD:C_0805_2012Metric, F.Cu at (149.7, 84.0)
- added J3: Conn_01x02_Socket, Resistor_SMD:R_0805_2012Metric, F.Cu at (154.2, 84.4)
- added R10: 2k, Resistor_SMD:R_0805_2012Metric, F.Cu at (154.2, 90.3)
- added R9: 10k, Resistor_SMD:R_0805_2012Metric, F.Cu at (154.2, 87.4)
- added SW4: SW_Push, Button_Switch_THT:SW_PUSH_6mm, F.Cu at (110.0, 82.3)
- added SW5: SW_SPDT, Button_Switch_THT:SW_Slide_SPDT_Straight_CK_OS102011MS2Q, F.Cu at (155.9, 80.0)
- added U5: MCP73831-2-OT, Package_TO_SOT_SMD:SOT-23-5, F.Cu at (121.1, 82.7)
- added U6: SCD40-D-R2, Sensor:Sensirion_SCD4x-1EP_10.1x10.1mm_P1.25mm_EP4.8x4.8mm, F.Cu at (114.2, 74.4)
Connections:
- J1 pad A4: +5V -> /USB_IN
- J1 pad A6: /IO18 -> /IO19
- J1 pad A7: /IO19 -> /IO18
- J1 pad A9: +5V -> /USB_IN
- J1 pad B4: +5V -> /USB_IN
- J1 pad B6: /IO18 -> /IO19
- J1 pad B7: /IO19 -> /IO18
- J1 pad B9: +5V -> /USB_IN
- U1 pad 3: /IO4 -> /Read_User
- U2 pad 1: +5V -> /VSYS
- U2 pad 3: +5V -> /VSYS

Commit message: Initial commit for air quality sensor
Parts:
- removed the C4 at (32.5, 41.0)
- removed D2: LED, LED_SMD:LED_0805_2012Metric
- removed the R9 at (67.5, 53.0)
- J3: value Conn_01x02_Socket -> Batt terminal
- moved SW5 146.0 mm to (24.5, 16.5)
- moved J3 145.8 mm to (21.0, 25.0), turned to -90 degrees
- moved R10 128.5 mm to (33.6, 46.0), turned to 180 degrees
- moved C4 127.2 mm to (33.0, 27.5), turned to 180 degrees
- moved C9 124.1 mm to (34.5, 38.0), turned to -90 degrees
- moved C10 119.6 mm to (40.5, 38.5)
- moved R9 116.8 mm to (51.1, 32.5)
- moved U5 90.4 mm to (39.4, 44.0), turned to 180 degrees
- moved C8 80.0 mm to (72.0, 62.0), turned to -90 degrees
- moved C11 67.1 mm to (100.5, 44.5)
- moved SW4 54.6 mm to (60.2, 59.8)
- moved C7 37.3 mm to (108.7, 38.8)
- moved U3 36.1 mm to (80.0, 56.0)
- moved U4 35.9 mm to (113.7, 38.8)
- moved C6 35.2 mm to (83.5, 56.0)
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Routing:
- net +3.3V: track 144.0 -> 0.00 mm, vias 2 -> 0
- net /I2C_SCL: track 113.0 -> 0.00 mm, vias 5 -> 0
- net /EN: track 69.4 -> 0.00 mm, vias 2 -> 0
- net /I2C_SDA: track 68.4 -> 0.00 mm, vias 4 -> 0
- net /BOOT: track 51.4 -> 0.00 mm, vias 2 -> 0
- net /USER_SW: track 44.3 -> 0.00 mm
- net /IO4: track 34.0 -> 0.00 mm, vias 6 -> 0
- net /IO19: track 23.1 -> 0.00 mm, vias 2 -> 0
- net +5V: track 21.0 -> 0.00 mm
- net Net-(J1-CC1): track 17.6 -> 0.00 mm
- net Net-(J1-CC2): track 15.1 -> 0.00 mm
- net GND: track 13.2 -> 0.00 mm
- net Net-(D1-A): track 2.06 -> 0.00 mm
